File: Design Files/Cap Bank V1/Passive Cap Bank V1/Passive Cap Bank V1.kicad_sch (KiCad schematic)
At the start: 29 parts, among them J1 XT30-Male, Q1 BC817-40, Q2 BC817-40, Q3 BC817-40, Q4 BC817-40, Q5 BC817-40, Q6 BC817-40, SW1 SW_Push_Open

Commit message: Started Layout
Parts:
- removed J1: XT30-Male, PassiveBankV1:XT30PW-M, symbol Connector:Conn_01x02_Pin
- added J2: XT30PW-M, XT30PW-M:AMASS_XT30PW-M, symbol PassiveBankV1:XT30PW-M
Connections:
- net GND: now also J2.N
- net V_15: now also J2.P
Changed lines of the file:
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@@
 	(wire
 		(pts
-			(xy 97.79 34.29) (xy 92.71 34.29)
+			(xy 102.87 35.56) (xy 97.79 35.56)
 		)
 		(stroke
@@
 	(wire
 		(pts
-			(xy 97.79 31.75) (xy 97.79 34.29)
+			(xy 102.87 33.02) (xy 102.87 35.56)
 		)
 		(stroke
@@
 	(wire
 		(pts
-			(xy 97.79 36.83) (xy 97.79 39.37)
+			(xy 102.87 38.1) (xy 102.87 40.64)
 		)
 		(stroke
@@
 	(wire
 		(pts
-			(xy 92.71 36.83) (xy 97.79 36.83)
+			(xy 97.79 38.1) (xy 102.87 38.1)
 		)
 		(stroke
@@
 	(symbol
 		(lib_id "power:VCC")
-		(at 97.79 31.75 0)
+		(at 102.87 33.02 0)
 		(unit 1)
 		(exclude_from_sim no)
@@
 		(fields_autoplaced yes)
 		(property "Reference" "#PWR03"
-			(at 97.79 35.56 0)
+			(at 102.87 36.83 0)
 			(effects
 				(font
@@
 		)
 		(property "Value" "V_15"
-			(at 97.79 26.67 0)
+			(at 102.87 27.94 0)
 			(effects
 				(font
@@
 		)
 		(property "Footprint" ""
-			(at 97.79 31.75 0)
+			(at 102.87 33.02 0)
 			(effects
 				(font
@@
 		)
 		(property "Datasheet" ""
-			(at 97.79 31.75 0)
+			(at 102.87 33.02 0)
 			(effects
 				(font
@@
 		)
 		(property "Description" "Power symbol creates a global label with name \"VCC\""
-			(at 97.79 31.75 0)
+			(at 102.87 33.02 0)
 			(effects
 				(font
@@
 	)
 	(symbol
+		(lib_id "PassiveBankV1:XT30PW-M")
+		(at 92.71 35.56 0)
+		(unit 1)
+		(exclude_from_sim no)
+		(in_bom yes)
+		(on_board yes)
+		(dnp no)
+		(fields_autoplaced yes)
+		(property "Reference" "J2"
+			(at 88.9 27.94 0)
+			(effects
+				(font
+					(size 1.27 1.27)
+				)
+			)
+		)
+		(property "Value" "XT30PW-M"
+			(at 88.9 30.48 0)
+			(effects
+				(font
+					(size 1.27 1.27)
+				)
+			)
+		)
+		(property "Footprint" "XT30PW-M:AMASS_XT30PW-M"
+			(at 93.218 20.574 0)
+			(effects
+				(font
+					(size 1.27 1.27)
+				)
+				(justify bottom)
+				(hide yes)
+			)
+		)
+		(property "Datasheet" ""
+			(at 92.71 35.56 0)
+			(effects
+				(font
+					(size 1.27 1.27)
+				)
+				(hide yes)
+			)
+		)
+		(property "Description" ""
+			(at 92.71 35.56 0)
+			(effects
+				(font
+					(size 1.27 1.27)
+				)
+				(hide yes)
+			)
+		)
+		(property "MF" "AMASS"
+			(at 74.93 41.402 0)
+			(effects
+				(font
+					(size 1.27 1.27)
+				)
+				(justify bottom)
+				(hide yes)
+			)
+		)
+		(property "MAXIMUM_PACKAGE_HEIGHT" "5 mm"
+			(at 75.438 39.624 0)
+			(effects
+				(font
+					(size 1.27 1.27)
+				)
+				(justify bottom)
+				(hide yes)
+			)
+		)
+		(property "Package" "None"
+			(at 73.914 34.29 0)
+			(effects
+				(font
+					(size 1.27 1.27)
+				)
+				(justify bottom)
+				(hide yes)
+			)
+		)
+		(property "Price" "None"
+			(at 74.422 44.45 0)
+			(effects
+				(font
+					(size 1.27 1.27)
+				)
+				(justify bottom)
+				(hide yes)
+			)
+		)
+		(property "Check_prices" "https://www.snapeda.com/parts/XT30PW-M/AMASS/view-part/?ref=eda"
+			(at 93.726 23.622 0)
+			(effects
+				(font
+					(size 1.27 1.27)
+				)
+				(justify bottom)
+				(hide yes)
+			)
+		)
+		(property "STANDARD" "Manufacturer Recommendations"
+			(at 91.694 18.288 0)
+			(effects
+				(font
+					(size 1.27 1.27)
+				)
+				(justify bottom)
+				(hide yes)
+			)
+		)
+		(property "PARTREV" "1.2"
+			(at 72.898 32.004 0)
+			(effects
+				(font
+					(size 1.27 1.27)
+				)
+				(justify bottom)
+				(hide yes)
+			)
+		)
+		(property "SnapEDA_Link" "https://www.snapeda.com/parts/XT30PW-M/AMASS/view-part/?ref=snap"
+			(at 92.964 26.924 0)
+			(effects
+				(font
+					(size 1.27 1.27)
+				)
+				(justify bottom)
+				(hide yes)
+			)
+		)
+		(property "MP" "XT30PW-M"
+			(at 115.062 34.544 0)
+			(effects
+				(font
+					(size 1.27 1.27)
+				)
+				(justify bottom)
+				(hide yes)
+			)
+		)
+		(property "Description_1" "\nSocket; DC supply; XT30; male; PIN: 2; on PCBs; THT; Colour: yellow\n"
+			(at 92.71 48.514 0)
+			(effects
+				(font
+					(size 1.27 1.27)
+				)
+				(justify bottom)
+				(hide yes)
+			)
+		)
+		(property "MANUFACTURER" "Amass"
+			(at 74.422 36.322 0)
+			(effects
+				(font
+					(size 1.27 1.27)
+				)
+				(justify bottom)
+				(hide yes)
+			)
+		)
+		(property "Availability" "Not in stock"
+			(at 110.744 31.242 0)
+			(effects
+				(font
+					(size 1.27 1.27)
+				)
+				(justify bottom)
+				(hide yes)
+			)
+		)
+		(property "SNAPEDA_PN" "XT30PW-M"
+			(at 117.856 40.132 0)
+			(effects
+				(font
+					(size 1.27 1.27)
+				)
+				(justify bottom)
+				(hide yes)
+			)
+		)
+		(pin "P"
+		)
+		(pin "N"
+		)
+		(instances
+			(project ""
+				(path "/6fc4e927-9d0e-48ab-aaa4-774eb70de429"
+					(reference "J2")
+					(unit 1)
+				)
+			)
+		)
+	)
+	(symbol
 		(lib_id "PCM_Generic:C,IEC")
 		(at 151.13 57.15 0)
@@
 	(symbol
 		(lib_id "power:GND")
-		(at 97.79 39.37 0)
+		(at 102.87 40.64 0)
 		(unit 1)
 		(exclude_from_sim no)
@@
 		(fields_autoplaced yes)
 		(property "Reference" "#PWR04"
-			(at 97.79 45.72 0)
+			(at 102.87 46.99 0)
 			(effects
 				(font
@@
 		)
 		(property "Value" "GND"
-			(at 97.79 44.45 0)
+			(at 102.87 45.72 0)
 			(effects
 				(font
@@
 		)
 		(property "Footprint" ""
-			(at 97.79 39.37 0)
+			(at 102.87 40.64 0)
 			(effects
 				(font
@@
 		)
 		(property "Datasheet" ""
-			(at 97.79 39.37 0)
+			(at 102.87 40.64 0)
 			(effects
 				(font
@@
 		)
 		(property "Description" "Power symbol creates a global label with name \"GND\" , ground"
-			(at 97.79 39.37 0)
+			(at 102.87 40.64 0)
 			(effects
 				(font
@@
 					(unit 1)
 				)
-			)
-		)
-	)
-	(symbol
-		(lib_id "Connector:Conn_01x02_Pin")
-		(at 87.63 34.29 0)
-		(unit 1)
-		(exclude_from_sim no)
-		(in_bom yes)
-		(on_board yes)
-		(dnp no)
-		(property "Reference" "J1"
-			(at 85.598 35.56 0)
-			(effects
-				(font
-					(size 1.27 1.27)
-				)
-			)
-		)
-		(property "Value" "XT30-Male"
-			(at 86.614 39.624 0)
-			(effects
-				(font
-					(size 1.27 1.27)
-				)
-			)
-		)
-		(property "Footprint" "PassiveBankV1:XT30PW-M"
-			(at 87.63 34.29 0)
-			(effects
-				(font
-					(size 1.27 1.27)
-				)
-				(hide yes)
-			)
-		)
-		(property "Datasheet" "~"
-			(at 87.63 34.29 0)
-			(effects
-				(font
-					(size 1.27 1.27)
-				)
-				(hide yes)
-			)
-		)
-		(property "Description" "Generic connector, single row, 01x02, script generated"
-			(at 87.63 34.29 0)
-			(effects
-				(font
-					(size 1.27 1.27)
-				)
-				(hide yes)
-			)
-		)
-		(pin "1"
-		)
-		(pin "2"
-		)
-		(instances
-			(project ""
-				(path "/6fc4e927-9d0e-48ab-aaa4-774eb70de429"
-					(reference "J1")
-					(unit 1)
-				)
