File: Design Files/Cap Bank V1/Passive Cap Bank V1/_autosave-Passive Cap Bank V1.kicad_pcb (KiCad board)
At the start: 2 copper layers, 29 parts, among them J1 XT30-Male, Q1 BC817-40, Q2 BC817-40, Q3 BC817-40, Q4 BC817-40, Q5 BC817-40, Q6 BC817-40, SW1 SW_Push_Open

Commit message: Started Layout
Parts:
- moved R13 200.8 mm to (140.0, 124.0)
- moved D1 172.7 mm to (160.3, 154.0), turned to 90 degrees
Changed lines of the file:
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@@
 	(footprint "PassiveBankV1:10mm LED"
 		(layer "F.Cu")
-		(at 325.41 103.12)
+		(at 160.335012 153.985012 90)
 		(tags "WP813SURDK ")
 		(property "Reference" "D1"
-			(at 0 -6.5 0)
+			(at 0 -6.5 90)
 			(unlocked yes)
 			(layer "F.SilkS")
@@
 		)
 		(property "Value" "10mm_LED"
-			(at 0 6.5 0)
+			(at 0 6.5 90)
 			(unlocked yes)
 			(layer "F.Fab")
@@
 		)
 		(property "Footprint" "PassiveBankV1:10mm LED"
-			(at -1.331012 -0.061012 0)
+			(at -1.331012 -0.061012 90)
 			(layer "F.Fab")
 			(hide yes)
@@
 		)
 		(property "Datasheet" ""
-			(at -1.331012 -0.061012 0)
+			(at -1.331012 -0.061012 90)
 			(layer "F.Fab")
 			(hide yes)
@@
 		)
 		(property "Description" "Light emitting diode"
-			(at -1.331012 -0.061012 0)
+			(at -1.331012 -0.061012 90)
 			(layer "F.Fab")
 			(hide yes)
@@
 		(attr through_hole)
 		(fp_line
+			(start -6.195112 -0.696012)
+			(end -6.195112 0.573988)
+			(stroke
+				(width 0.1524)
+				(type solid)
+			)
+			(layer "F.SilkS")
+		)
+		(fp_line
 			(start -6.957112 -0.696012)
 			(end -6.957112 0.573988)
@@
 		)
 		(fp_line
+			(start -5.941112 -0.061012)
+			(end -7.211112 -0.061012)
+			(stroke
+				(width 0.1524)
+				(type solid)
+			)
+			(layer "F.SilkS")
+		)
+		(fp_line
 			(start -6.957112 -0.061012)
 			(end -6.195112 -0.696012)
@@
 			(layer "F.SilkS")
 		)
-		(fp_line
-			(start -6.195112 -0.696012)
-			(end -6.195112 0.573988)
+		(fp_circle
+			(center -0.061012 -0.061012)
+			(end 5.565088 -0.061012)
 			(stroke
 				(width 0.1524)
 				(type solid)
 			)
+			(fill none)
 			(layer "F.SilkS")
 		)
 		(fp_line
-			(start -5.941112 -0.061012)
-			(end -7.211112 -0.061012)
-			(stroke
-				(width 0.1524)
-				(type solid)
-			)
-			(layer "F.SilkS")
-		)
-		(fp_circle
-			(center -0.061012 -0.061012)
-			(end 5.565088 -0.061012)
+			(start 2.307911 -5.814112)
+			(end 5.692088 -2.429935)
 			(stroke
-				(width 0.1524)
+				(width 0.0254)
 				(type solid)
 			)
-			(fill none)
-			(layer "F.SilkS")
+			(layer "F.CrtYd")
 		)
 		(fp_line
-			(start -5.814112 -2.429935)
-			(end -2.429935 -5.814112)
+			(start -2.429935 -5.814112)
+			(end 2.307911 -5.814112)
 			(stroke
 				(width 0.0254)
@@
 		)
 		(fp_line
-			(start -5.814112 2.307911)
-			(end -5.814112 -2.429935)
+			(start 5.692088 -2.429935)
+			(end 5.692088 2.307911)
 			(stroke
 				(width 0.0254)
@@
 		)
 		(fp_line
-			(start -2.429935 -5.814112)
-			(end 2.307911 -5.814112)
+			(start -5.814112 -2.429935)
+			(end -2.429935 -5.814112)
 			(stroke
 				(width 0.0254)
@@
 		)
 		(fp_line
-			(start -2.429935 5.692088)
-			(end -5.814112 2.307911)
+			(start 5.692088 2.307911)
+			(end 2.307911 5.692088)
 			(stroke
 				(width 0.0254)
@@
 		)
 		(fp_line
-			(start 2.307911 -5.814112)
-			(end 5.692088 -2.429935)
+			(start -5.814112 2.307911)
+			(end -5.814112 -2.429935)
 			(stroke
 				(width 0.0254)
@@
 		)
 		(fp_line
-			(start 5.692088 -2.429935)
-			(end 5.692088 2.307911)
+			(start -2.429935 5.692088)
+			(end -5.814112 2.307911)
 			(stroke
 				(width 0.0254)
@@
 		)
 		(fp_line
-			(start 5.692088 2.307911)
-			(end 2.307911 5.692088)
+			(start -6.195112 -0.696012)
+			(end -6.195112 0.573988)
 			(stroke
 				(width 0.0254)
 				(type solid)
 			)
-			(layer "F.CrtYd")
+			(layer "F.Fab")
 		)
 		(fp_line
@@
 		)
 		(fp_line
+			(start -5.941112 -0.061012)
+			(end -7.211112 -0.061012)
+			(stroke
+				(width 0.0254)
+				(type solid)
+			)
+			(layer "F.Fab")
+		)
+		(fp_line
 			(start -6.957112 -0.061012)
 			(end -6.195112 -0.696012)
@@
 			(layer "F.Fab")
 		)
-		(fp_line
-			(start -6.195112 -0.696012)
-			(end -6.195112 0.573988)
-			(stroke
-				(width 0.0254)
-				(type solid)
-			)
-			(layer "F.Fab")
-		)
-		(fp_line
-			(start -5.941112 -0.061012)
-			(end -7.211112 -0.061012)
-			(stroke
-				(width 0.0254)
-				(type solid)
-			)
-			(layer "F.Fab")
-		)
 		(fp_circle
 			(center -0.061012 -0.061012)
@@
 		)
 		(pad "1" thru_hole rect
-			(at -1.331012 -0.061012)
+			(at -1.331012 -0.061012 90)
 			(size 1.397 1.397)
 			(drill 0.889)
@@
 		)
 		(pad "2" thru_hole circle
-			(at 1.208988 -0.061012)
+			(at 1.208988 -0.061012 90)
 			(size 1.397 1.397)
 			(drill 0.889)
@@
 	(footprint "PassiveBankV1:100Watt2"
 		(layer "F.Cu")
-		(at 336.41 82.62)
+		(at 139.955 123.952)
 		(tags "TEH100M2R00FE ")
 		(property "Reference" "R13"
@@
 	)
 	(gr_rect
-		(start 317.81 9.93)
-		(end 373.81 37.93)
+		(start 220.218 56.388)
+		(end 276.218 84.388)
 		(stroke
 			(width 0.1)
