File: Design Files/Cap Bank V1/Passive Cap Bank V1/_autosave-Passive Cap Bank V1.kicad_pcb (KiCad board)
At the start: 2 copper layers, 76 x 120 mm, 30 parts, among them J1 XT30-Male, Q1 BC817-40, Q2 BC817-40, Q3 BC817-40, Q4 BC817-40, Q5 BC817-40, Q6 BC817-40, SW1 SW_Push_Open

Commit message: supercap boad layout back maybe change
title
Parts:
- moved SW1 49.7 mm to (188.7, 58.1), turned to -90 degrees
- moved R13 29.7 mm to (157.5, 49.2), turned to 90 degrees
- moved D1 17.4 mm to (169.1, 50.6), turned to 180 degrees
- moved R14 14.1 mm to (170.4, 42.7), turned to 180 degrees
Routing:
- net Net-(D1-A): track 1.71 -> 0.00 mm
Other:
- board size 76 x 120 mm -> 76 x 122 mm
