File: Design Files/Cap Bank V1/Passive Cap Bank V1/Passive Cap Bank V1.kicad_pcb (KiCad board)
At the start: 2 copper layers, 29 parts, among them J1 XT30-Male, Q1 BC817-40, Q2 BC817-40, Q3 BC817-40, Q4 BC817-40, Q5 BC817-40, Q6 BC817-40, SW1 SW_Push_Open

Commit message: Layout and Routing Progress
Parts:
- moved R6 312.4 mm to (135.1, 114.5), turned to 0 degrees
- moved R5 307.9 mm to (135.1, 106.0), turned to 180 degrees
- moved Q3 306.3 mm to (137.1, 110.6), turned to -90 degrees
- moved R4 303.6 mm to (134.9, 94.0), turned to 0 degrees
- moved R3 301.3 mm to (135.1, 85.5), turned to 180 degrees
- moved R1 299.1 mm to (135.4, 66.0), turned to 180 degrees
- moved R2 299.1 mm to (135.4, 74.5), turned to 0 degrees
- moved Q2 298.5 mm to (137.0, 90.1), turned to -90 degrees
- moved Q1 294.9 mm to (137.5, 70.5), turned to -90 degrees
- moved C3 281.9 mm to (150.0, 111.3), turned to -90 degrees
- moved C2 273.1 mm to (150.0, 91.3), turned to -90 degrees
- moved C1 269.9 mm to (150.0, 71.3), turned to -90 degrees
- moved C4 253.5 mm to (168.5, 120.7), turned to 90 degrees
- moved C5 240.5 mm to (168.5, 100.7), turned to 90 degrees
- moved C6 233.8 mm to (168.5, 80.8), turned to 90 degrees
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Routing:
- net GND: track 15.7 -> 84.4 mm
- net Net-(D1-A): track 0.00 -> 61.7 mm
- net V_15: track 15.4 -> 63.4 mm
- net Net-(D1-K): track 0.00 -> 13.3 mm
Other:
- board outline added: 76 x 144 mm
- board text added: "CAN-F Ref System"
- board text added: "Cap Management Module"
- board text added: "XT30-F Power In/Out"
- board text added: "XT30-F Pre-Inspection"
- board text added: "XT30-M Cap Bank"

Commit message: Routing done. Luci is amazing
Other:
- board text added: "Do NOT EXCEED: 7A or 15V YOU WILL BLOW UP A TRACE OR A CAPACITOR"
- board text added: "Negative"
- board text added: "Positive"
Changed lines of the file:
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@@
 		(tags "TEH100M2R00FE ")
 		(property "Reference" "R13"
-			(at 0 -4.5 0)
+			(at 0 0 0)
 			(unlocked yes)
 			(layer "F.SilkS")
@@
 		(at 173 63 -90)
 		(property "Reference" "J1"
-			(at 0 -4 90)
+			(at 0 7.5 90)
 			(layer "F.SilkS")
 			(effects
@@
 		)
 	)
-	(gr_rect
-		(start 169 34)
-		(end 196.5 55)
-		(stroke
-			(width 0.05)
+	(gr_poly
+		(pts
+			(xy 169 34) (xy 196.5 34) (xy 196.5 51.5) (xy 196.5 73) (xy 178.5 73) (xy 178.5 55) (xy 169 55)
+		)
+		(stroke
+			(width 0.1)
 			(type solid)
 		)
@@
 		(fill none)
 		(layer "F.SilkS")
+	)
+	(gr_rect
+		(start 169 34)
+		(end 186 55)
+		(stroke
+			(width 0.05)
+			(type solid)
+		)
+		(fill solid)
+		(layer "F.Mask")
 	)
 	(gr_circle
@@
 		(fill none)
 		(layer "Edge.Cuts")
+	)
+	(gr_text "Positive"
+		(at 177 62 90)
+		(layer "F.SilkS")
+		(effects
+			(font
+				(size 0.5 0.5)
+				(thickness 0.1)
+			)
+			(justify left bottom)
+		)
 	)
 	(gr_text "CAN-F\nRef System"
@@
 		)
 	)
+	(gr_text "Negative"
+		(at 177 67.5 90)
+		(layer "F.SilkS")
+		(effects
+			(font
+				(size 0.5 0.5)
+				(thickness 0.1)
+			)
+			(justify left bottom)
+		)
+	)
+	(gr_text "Do NOT EXCEED:\n7A or 15V\nYOU WILL BLOW UP A\nTRACE OR A CAPACITOR"
+		(at 187.5 66 0)
+		(layer "F.SilkS")
+		(effects
+			(font
+				(size 1 1)
+				(thickness 0.1)
+			)
+			(justify bottom)
+		)
+	)

Commit message: Minor Changes. Added Logo and warnings
Parts:
- added G***: LOGO, PassiveBankV1:10mm RM Logo, F.Cu at (137.5, 123.0)
- moved R13 3.50 mm to (177.4, 27.0)
Routing:
- net Net-(D1-A): track 61.7 -> 59.0 mm
- net GND: track 84.4 -> 85.4 mm
Other:
- outline, holes or cut-outs redrawn
- board text added: "Caution! Area may be hot!"
- board text added: "DO NOT EXCEED: 7A or 15V YOU WILL BLOW UP A TRACE OR A CAPACITOR Use at your own risk"
- board text added: "Designed by Rose-Hulman Thornbots, October 2024 https://github.com/Thornbots/Supa-Cap Passive Cap Bank V1"
- board text added: "Ground"
- board text removed: "Do NOT EXCEED: 7A or 15V YOU WILL BLOW UP A TRACE OR A CAPACITOR"
- board text removed: "Negative"
