File: Design Files/Controller Board V1/5V_PSU.kicad_sch (KiCad schematic)
At the start: 8 parts, among them U1 LMR51420XDDCR

Commit message: here we go agane
Updating footprints and tackling general layout
Parts:
- Cinx1: footprint Capacitor_SMD:C_0603_1608Metric_Pad1.08x0.95mm_HandSolder -> Capacitor_SMD:C_0603_1608Metric
- L1: footprint NRS8030T100MJGJ:IND_TAIYO_NRS8030_TAY -> Library:IND_TAIYO_NRS8030_TAY
- U1: footprint LMR51420XDDCR:SOT95P280X110-6N -> Library:SOT23_DDC_TEX
Changed lines of the file:
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@@
 			)
 		)
-		(property "Footprint" "Capacitor_SMD:C_0603_1608Metric_Pad1.08x0.95mm_HandSolder"
+		(property "Footprint" "Capacitor_SMD:C_0603_1608Metric"
 			(at 119.5832 106.426 0)
 			(effects
@@
 			)
 		)
-		(property "Footprint" "NRS8030T100MJGJ:IND_TAIYO_NRS8030_TAY"
+		(property "Footprint" "Library:IND_TAIYO_NRS8030_TAY"
 			(at 181.864 87.376 0)
 			(effects
@@
 			)
 		)
-		(property "Footprint" "LMR51420XDDCR:SOT95P280X110-6N"
+		(property "Footprint" "Library:SOT23_DDC_TEX"
 			(at 142.24 84.836 0)
 			(effects
