File: Design Files/Controller Board V1/Control Board V1.kicad_pcb (KiCad board)
At the start: 2 copper layers, 75 x 125 mm, 36 parts, among them J1 XT30PW-M, J2 XT30PW-M, J3 XT30PW-M, J4 XT30PW-M, J5 XT30PW-M, J6 XT30PW-M, J7 XT30PW-F, J8 SM04B-GHS-TB_LF__SN_-, Q1 LMG5200, U1 LMR51420XDDCR

Commit message: Assigning footprints and ading to schematic
Parts:
- removed the J1 at (133.1, 59.2)
- removed the J1 at (109.2, 41.8)
- removed the REF** at (81.1, 46.6)
- added J1: XT30PW-F, PassiveBankV1:XT30PW-F, F.Cu at (110.4, 54.1)
- added R10: 10KΩ, Resistor_SMD:R_0603_1608Metric, F.Cu at (159.6, 51.2)
- added R11: 10KΩ, Resistor_SMD:R_0603_1608Metric, F.Cu at (159.6, 53.8)
- added R12: 10KΩ, Resistor_SMD:R_0603_1608Metric, F.Cu at (159.6, 56.3)
- added R2: 0.01Ω, Resistor_SMD:R_0805_2012Metric, F.Cu at (153.4, 41.9)
- added R3: 10KΩ, Resistor_SMD:R_0603_1608Metric, F.Cu at (153.2, 44.7)
- added R4: 10KΩ, Resistor_SMD:R_0603_1608Metric, F.Cu at (153.2, 47.2)
- added R5: 0.01Ω, Resistor_SMD:R_0805_2012Metric, F.Cu at (163.8, 41.9)
- added R6: 10KΩ, Resistor_SMD:R_0603_1608Metric, F.Cu at (159.6, 41.7)
- added R7: 10KΩ, Resistor_SMD:R_0603_1608Metric, F.Cu at (159.6, 44.2)
- added R8: 10KΩ, Resistor_SMD:R_0603_1608Metric, F.Cu at (159.6, 46.7)
- added R9: 0.01Ω, Resistor_SMD:R_0805_2012Metric, F.Cu at (163.8, 51.5)
- added U5: SC0917, Module:RaspberryPi_Pico_Common_THT, F.Cu at (80.9, 43.8)
- J2, J4, J6: footprint XT30PW-M:AMASS_XT30PW-M -> PassiveBankV1:XT30PW-M; moved to F.Cu
- J3, J5: footprint XT30PW-M:AMASS_XT30PW-M -> PassiveBankV1:XT30PW-M
- J7: value XT30PW-F -> XT30PW-M; footprint XT30PW-F:AMASS_XT30PW-F -> PassiveBankV1:XT30PW-M; moved to B.Cu
- moved J6 108.3 mm to (215.2, 23.0), turned to 0 degrees
- moved J5 93.2 mm to (200.3, 23.0), turned to 0 degrees
- moved J4 67.7 mm to (185.5, 23.0), turned to 0 degrees
- moved J3 62.9 mm to (170.6, 23.0), turned to 0 degrees
- moved J2 57.5 mm to (155.8, 23.0), turned to 0 degrees
- moved J7 7.41 mm to (110.4, 44.2), turned to 180 degrees
Connections:
- J2 pad S1: unconnected-(J2-PadS1) -> (no net)
- J2 pad S2: unconnected-(J2-PadS2) -> (no net)
- J3 pad S1: unconnected-(J3-PadS1) -> (no net)
- J3 pad S2: unconnected-(J3-PadS2) -> (no net)
- J4 pad S1: unconnected-(J4-PadS1) -> (no net)
- J4 pad S2: unconnected-(J4-PadS2) -> (no net)
- J5 pad S1: unconnected-(J5-PadS1) -> (no net)
- J5 pad S2: unconnected-(J5-PadS2) -> (no net)
- J6 pad S1: unconnected-(J6-PadS1) -> (no net)
- J6 pad S2: unconnected-(J6-PadS2) -> (no net)
- J7 pad S1: unconnected-(J7-PadS1) -> (no net)
- J7 pad S2: unconnected-(J7-PadS2) -> (no net)
- Q1 pad 1: /LMG5200/24V -> unconnected-(Q1-Pad1)
- Q1 pad 8: Net-(L2-Pad2) -> unconnected-(Q1-Pad8)
- Q1 pad 9: /LMG5200/GND -> unconnected-(Q1-Pad9)

Commit message: yay(meeting 2/16/2025)
Parts:
- moved J6 187.9 mm to (85.7, 159.2), turned to 180 degrees
- moved J5 168.9 mm to (100.5, 159.2), turned to 180 degrees
- moved J4 153.2 mm to (115.4, 159.2), turned to 180 degrees
- moved J3 63.7 mm to (133.6, 74.8), turned to -90 degrees
- moved J2 43.2 mm to (133.6, 60.0), turned to -90 degrees

Commit message: Major Schematic Progress
Parts:
- J4, J5, J6: moved to B.Cu
- moved J6 108.6 mm to (130.0, 60.1), turned to 90 degrees
- moved J5 89.3 mm to (130.0, 74.9), turned to 90 degrees
- moved J4 70.9 mm to (130.0, 89.8), turned to 90 degrees

Commit message: idk
drew a instead of getting the footprint
and tested potential layouts but idk yet
Parts:
- added R1: 39k, Resistor_SMD:R_0603_1608Metric, F.Cu at (178.7, 114.5)
- added R13: 2k, Resistor_SMD:R_0603_1608Metric, F.Cu at (178.7, 117.0)
- added R14: 2k, Resistor_SMD:R_0603_1608Metric, F.Cu at (178.7, 119.5)
- added R15: 11k, Resistor_SMD:R_0603_1608Metric, F.Cu at (178.7, 122.0)
- added R16: 0, Resistor_SMD:R_0603_1608Metric, F.Cu at (184.8, 114.5)
- added R17: 0, Resistor_SMD:R_0603_1608Metric, F.Cu at (184.8, 117.0)
- Cboot1, Cin1, Cinx1, Cout1, L1, R3, R4, Rfbb1, Rfbt1, U1: moved to B.Cu
- J4, J5, J6: moved to F.Cu
- moved Cinx1 117.7 mm to (89.2, 49.6), turned to 0 degrees
- moved Cin1 114.3 mm to (89.7, 51.6), turned to 0 degrees
- moved U1 110.6 mm to (88.6, 55.4), turned to 90 degrees
- moved Cboot1 109.8 mm to (86.4, 58.1), turned to -90 degrees
- moved Rfbb1 109.0 mm to (93.1, 52.0), turned to -90 degrees
- moved J6 108.4 mm to (85.3, 158.9), turned to 180 degrees
- moved Rfbt1 107.2 mm to (94.3, 52.0), turned to 90 degrees
- moved Cout1 103.6 mm to (92.9, 56.0), turned to 180 degrees
- moved L1 97.2 mm to (91.4, 62.1), turned to 0 degrees
- moved J5 89.1 mm to (100.1, 158.9), turned to 180 degrees
- moved J4 70.7 mm to (115.0, 158.9), turned to 180 degrees
- moved R3 51.1 mm to (104.8, 61.2)
- moved R4 50.8 mm to (104.8, 62.8)
- moved R2 46.3 mm to (113.0, 64.6), turned to 90 degrees
- moved Q1 21.3 mm to (173.2, 98.2)
Connections:
- net /5V_PSU/VIN renamed 24V
- Cin1 pad 2: /5V_PSU/GND -> P_GND
- Cinx1 pad 2: /5V_PSU/GND -> P_GND
- Cout1 pad 1: /5V_PSU/IOUT -> 5V
- Cout1 pad 2: /5V_PSU/GND -> D_GND
- J1 pad N: unconnected-(J1-PadN) -> P_GND
- J1 pad P: unconnected-(J1-PadP) -> /CAP_IN
- J2 pad N: unconnected-(J2-PadN) -> P_GND
- J2 pad P: unconnected-(J2-PadP) -> /IO/24V_OUT
- J3 pad N: unconnected-(J3-PadN) -> P_GND
- J3 pad P: unconnected-(J3-PadP) -> /IO/24V_OUT
- J4 pad N: unconnected-(J4-PadN) -> P_GND
- J4 pad P: unconnected-(J4-PadP) -> /IO/24V_OUT
- J5 pad N: unconnected-(J5-PadN) -> P_GND
- J5 pad P: unconnected-(J5-PadP) -> /IO/24V_OUT
- J6 pad N: unconnected-(J6-PadN) -> P_GND
- J6 pad P: unconnected-(J6-PadP) -> /IO/24V_OUT
- J7 pad N: unconnected-(J7-PadN) -> P_GND
- J7 pad P: unconnected-(J7-PadP) -> /IO/24_IN_PMM
- J8 pad 1: unconnected-(J8-Pad1) -> /IO/I2C_TypeC_SDA
- J8 pad 2: unconnected-(J8-Pad2) -> D_GND
- J8 pad 3: unconnected-(J8-Pad3) -> /IO/I2C_TypeC_SCL
- J8 pad 4: unconnected-(J8-Pad4) -> D_GND
- J8 pad SH1: Net-(J8-SHIELD-PadSH1) -> unconnected-(J8-SHIELD-PadSH1)_0
- J8 pad SH2: Net-(J8-SHIELD-PadSH1) -> unconnected-(J8-SHIELD-PadSH1)
- Q1 pad 1: unconnected-(Q1-Pad1) -> /LMG5200/high_side_FET
- Q1 pad 2: unconnected-(Q1-HB-Pad2) -> Net-(Q1-HB)
- Q1 pad 3: unconnected-(Q1-HS-Pad3) -> Net-(Q1-HS)
- Q1 pad 4: /LMG5200/PWM_top -> /PWM_top
- Q1 pad 5: /LMG5200/PWM_bottom -> /PWM_bottom
- Q1 pad 6: /LMG5200/5V -> 5V
- Q1 pad 7: /LMG5200/sig-gnd -> D_GND
- Q1 pad 8: unconnected-(Q1-Pad8) -> Net-(L2-Pad1)
- Q1 pad 9: unconnected-(Q1-Pad9) -> P_GND
- R2 pad 1: /current_sensor1/VIN+ -> /CAP_IN
- R2 pad 2: /current_sensor1/VIN- -> /cap_volt
- R3 pad 1: /current_sensor1/3V3 -> 3.3V
- R3 pad 2: /current_sensor1/SCL -> /I2C_current_SCL
- R4 pad 1: /current_sensor1/3V3 -> 3.3V
- R4 pad 2: /current_sensor1/SDA -> /I2C_current_SDA
- Rfbb1 pad 2: /5V_PSU/GND -> D_GND
- Rfbt1 pad 1: /5V_PSU/IOUT -> 5V
- U5 pad 1: unconnected-(U5-GP0-Pad1) -> /IO/I2C_TypeC_SDA
- U5 pad 10: unconnected-(U5-GP7-Pad10) -> /Pico/LED4
- U5 pad 11: unconnected-(U5-GP8-Pad11) -> /IO/GPIO_3
- U5 pad 12: unconnected-(U5-GP9-Pad12) -> /IO/GPIO_2
- U5 pad 13: unconnected-(U5-GND__2-Pad13) -> GNDD
- U5 pad 14: unconnected-(U5-GP10-Pad14) -> /Pico/LED3
- U5 pad 15: unconnected-(U5-GP11-Pad15) -> /Pico/LED2
- U5 pad 16: unconnected-(U5-GP12-Pad16) -> /IO/GPIO_1
- U5 pad 17: unconnected-(U5-GP13-Pad17) -> /IO/GPIO_0
- U5 pad 18: unconnected-(U5-GND__3-Pad18) -> GNDD
- U5 pad 19: unconnected-(U5-GP14-Pad19) -> /Pico/LED1
- U5 pad 2: unconnected-(U5-GP1-Pad2) -> /IO/I2C_TypeC_SCL
- U5 pad 20: unconnected-(U5-GP15-Pad20) -> /Pico/LED0
- U5 pad 21: unconnected-(U5-GP16-Pad21) -> /PWM_bottom
- U5 pad 22: unconnected-(U5-GP17-Pad22) -> /PWM_top
- U5 pad 23: unconnected-(U5-GND__4-Pad23) -> GNDD
- U5 pad 24: /Pico/SCL -> /I2C_current_SCL
- U5 pad 25: /Pico/SDA -> /I2C_current_SDA
- U5 pad 28: unconnected-(U5-GND__5-Pad28) -> GNDD
- U5 pad 3: unconnected-(U5-GND-Pad3) -> GNDD
- U5 pad 31: unconnected-(U5-GP26-Pad31) -> /Pico/ADC_0
- U5 pad 32: unconnected-(U5-GP27-Pad32) -> /Pico/ADC_1
- U5 pad 33: unconnected-(U5-AGND-Pad33) -> GNDA
- U5 pad 34: unconnected-(U5-GP28-Pad34) -> /Pico/ADC_2
- U5 pad 36: /Pico/3.3V -> 3.3V
- U5 pad 38: unconnected-(U5-GND__6-Pad38) -> GNDD
- U5 pad 39: /Pico/5V -> 5V
- U5 pad 4: unconnected-(U5-GP2-Pad4) -> /Pico/LED7
- U5 pad 5: unconnected-(U5-GP3-Pad5) -> /Pico/LED6
- U5 pad 6: unconnected-(U5-GP4-Pad6) -> /IO/GPIO_5
- U5 pad 7: unconnected-(U5-GP5-Pad7) -> /IO/GPIO_4
- U5 pad 8: unconnected-(U5-GND__1-Pad8) -> GNDD
- U5 pad 9: unconnected-(U5-GP6-Pad9) -> /Pico/LED5
Other:
- board text added: "INA219"

Commit message: here we go agane
Updating footprints and tackling general layout
Parts:
- removed the Cboot1 at (86.4, 58.1)
- removed the Cin1 at (89.7, 51.6)
- removed the Cinx1 at (89.2, 49.6)
- removed the Cout1 at (92.9, 56.0)
- removed the Rfbb1 at (93.1, 52.0)
- removed the Rfbt1 at (94.3, 52.0)
- added C4: 100 nF, Capacitor_SMD:C_0603_1608Metric, B.Cu at (111.8, 62.9)
- added C5: 100 nF, Capacitor_SMD:C_0603_1608Metric, F.Cu at (190.1, 81.5)
- added C6: 100 nF, Capacitor_SMD:C_0603_1608Metric, F.Cu at (190.1, 86.0)
- added U2: INA219BIDR, Library:INA219, B.Cu at (107.2, 64.2)
- added U3: INA219BIDR, Library:INA219, F.Cu at (157.5, 78.2)
- added U4: INA219BIDR, Library:INA219, F.Cu at (162.8, 72.2)
- Cboot1, Cin1, Cout1, Q1, Rfbb1, Rfbt1: moved to B.Cu
- Cinx1: footprint Capacitor_SMD:C_0603_1608Metric_Pad1.08x0.95mm_HandSolder -> Capacitor_SMD:C_0603_1608Metric; moved to B.Cu
- moved Cinx1 93.4 mm to (88.1, 51.3)
- moved Cboot1 93.0 mm to (85.2, 59.8), turned to -90 degrees
- moved Rfbt1 90.0 mm to (93.2, 53.7), turned to 90 degrees
- moved R15 89.5 mm to (107.5, 67.8), turned to 180 degrees
- moved Rfbb1 89.5 mm to (92.0, 53.6), turned to 90 degrees
- moved Cin1 87.0 mm to (88.6, 53.3)
- moved Cout1 84.4 mm to (91.8, 57.6), turned to 180 degrees
- moved R1 82.4 mm to (110.9, 67.8), turned to 180 degrees
- moved Q1 65.0 mm to (109.2, 86.5), turned to 180 degrees
- moved R2 3.12 mm to (115.8, 65.8), turned to -90 degrees
- moved R4 2.91 mm to (102.5, 64.5), turned to 90 degrees
- moved R3 2.35 mm to (102.5, 61.3), turned to -90 degrees
- moved L1 2.04 mm to (90.2, 63.8)
- moved U1 2.01 mm to (87.4, 57.0)
- turned R13 to 180 degrees
Connections:
- L1 pad 1: (no net) -> Net-(U1-SW)
- L1 pad 2: (no net) -> 5V
- U1 pad 1: (no net) -> P_GND
- U1 pad 2: (no net) -> Net-(U1-SW)
- U1 pad 3: (no net) -> 24V
- U1 pad 4: (no net) -> Net-(U1-FB)
- U1 pad 5: (no net) -> 24V
- U1 pad 6: (no net) -> Net-(U1-CB)
Routing:
- net (no net): track 33.3 -> 0.00 mm, vias 2 -> 0
- net Net-(U1-FB): track 0.00 -> 13.1 mm
- net Net-(U1-SW): track 0.00 -> 6.04 mm
- net Net-(U1-CB): track 0.00 -> 6.03 mm, vias 0 -> 2
- net 24V: track 0.00 -> 4.29 mm
- net P_GND: track 0.00 -> 3.20 mm
- net 5V: track 0.00 -> 0.64 mm
Other:
- board text added: "L2"
- board text removed: "INA219"

Commit message: the board
yayyyyyyyyy
Parts:
- added C2: 0.1u, Capacitor_SMD:C_0603_1608Metric, B.Cu at (105.9, 77.8)
- added C3: 0.1u, Capacitor_SMD:C_0603_1608Metric, B.Cu at (105.9, 85.8)
- C5, C6, R10, R11, R12, R13, R14, R5, R6, R7, R8, R9, U3, U4: moved to B.Cu
- moved R13 84.2 mm to (103.1, 80.0), turned to 90 degrees
- moved R14 83.6 mm to (103.1, 83.8), turned to -90 degrees
- moved C6 76.5 mm to (115.1, 71.2), turned to -90 degrees
- moved C5 72.6 mm to (117.8, 88.6)
- moved R6 69.2 mm to (115.7, 95.3), turned to -90 degrees
- moved R7 67.8 mm to (117.8, 97.6)
- moved R8 64.0 mm to (120.7, 97.6), turned to 180 degrees
- moved R5 61.0 mm to (120.3, 84.7), turned to 180 degrees
- moved R11 56.8 mm to (106.1, 72.9), turned to 90 degrees
- moved R10 56.6 mm to (106.1, 69.9), turned to -90 degrees
- moved R12 56.3 mm to (106.9, 76.2)
- moved U4 52.2 mm to (110.6, 72.7)
- moved R9 51.2 mm to (117.7, 73.9), turned to 90 degrees
- moved U3 41.1 mm to (119.2, 93.1), turned to 90 degrees
- moved L1 12.7 mm to (88.4, 51.2), turned to 180 degrees
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
Commit message: general layout revised
goodnight
Parts:
- added C1: 10u, Capacitor_SMD:C_0603_1608Metric, F.Cu at (104.6, 80.5)
- added C10: 10u, Capacitor_SMD:C_0603_1608Metric, F.Cu at (114.9, 153.3)
- added C11: 10u, Capacitor_SMD:C_0603_1608Metric, F.Cu at (72.6, 124.6)
- added C7: 10u, Capacitor_SMD:C_0603_1608Metric, F.Cu at (85.4, 153.3)
- added C8: 10u, Capacitor_SMD:C_0603_1608Metric, F.Cu at (95.2, 153.3)
- added C9: 10u, Capacitor_SMD:C_0603_1608Metric, F.Cu at (105.1, 153.3)
- added D1: LED, LED_SMD:LED_0603_1608Metric, F.Cu at (157.0, 89.0)
- added D2: LED, LED_SMD:LED_0603_1608Metric, F.Cu at (157.0, 91.6)
- added D3: LED, LED_SMD:LED_0603_1608Metric, F.Cu at (157.0, 94.2)
- added D4: LED, LED_SMD:LED_0603_1608Metric, F.Cu at (157.0, 96.7)
- added D5: LED, LED_SMD:LED_0603_1608Metric, F.Cu at (157.0, 99.3)
- added D6: LED, LED_SMD:LED_0603_1608Metric, F.Cu at (157.0, 101.9)
- added D7: LED, LED_SMD:LED_0603_1608Metric, F.Cu at (157.0, 104.5)
- added D8: LED, LED_SMD:LED_0603_1608Metric, F.Cu at (157.0, 107.1)
- added R18: R, LED_SMD:LED_0805_2012Metric, F.Cu at (152.8, 95.3)
- added R19: R, LED_SMD:LED_0805_2012Metric, F.Cu at (152.8, 98.3)
- added R20: R, LED_SMD:LED_0805_2012Metric, F.Cu at (152.8, 101.4)
- added R21: R, LED_SMD:LED_0805_2012Metric, F.Cu at (152.8, 104.4)
- added R22: R, LED_SMD:LED_0805_2012Metric, F.Cu at (152.8, 107.4)
- added R23: R, LED_SMD:LED_0805_2012Metric, F.Cu at (152.8, 110.5)
- C4, C5, C6, R10, R11, R12, R3, R4, R6, R7, R8, U2, U3, U4: moved to F.Cu
- J2, J3, J4, J5, J6: value XT30PW-M -> XT30UPB-M; footprint PassiveBankV1:XT30PW-M -> Connector_AMASS:AMASS_XT30UPB-M_1x02_P5.0mm_Vertical
- J7: value XT30PW-M -> XT30UPB-M; footprint PassiveBankV1:XT30PW-M -> Connector_AMASS:AMASS_XT30UPB-M_1x02_P5.0mm_Vertical; moved to F.Cu
- R1: value 39k -> R; footprint Resistor_SMD:R_0603_1608Metric -> LED_SMD:LED_0805_2012Metric
- R15: value 11k -> R; footprint Resistor_SMD:R_0603_1608Metric -> LED_SMD:LED_0805_2012Metric
- R2: footprint Resistor_SMD:R_0805_2012Metric -> Resistor_SMD:R_2512_6332Metric
- R5, R9: footprint Resistor_SMD:R_0805_2012Metric -> Resistor_SMD:R_2512_6332Metric; moved to F.Cu
- moved J2 109.5 mm to (80.5, 155.8), turned to 90 degrees
- moved J7 93.3 mm to (67.3, 126.9), turned to 90 degrees
- moved J3 91.8 mm to (90.3, 155.8), turned to 90 degrees
- moved R5 59.3 mm to (73.6, 121.3)
- moved R9 57.8 mm to (94.3, 126.7)
- moved C5 57.2 mm to (68.4, 117.6)
- moved Cboot1 53.8 mm to (88.1, 108.8), turned to 0 degrees
- moved C6 53.6 mm to (97.0, 121.7)
- moved U3 53.3 mm to (69.8, 113.1), turned to -90 degrees
- moved L1 52.7 mm to (92.1, 103.8), turned to 90 degrees
- moved R6 51.8 mm to (66.3, 110.9), turned to 90 degrees
- moved U4 51.2 mm to (101.5, 123.1), turned to 180 degrees
- moved R7 50.6 mm to (68.4, 108.6)
- moved R8 50.6 mm to (71.3, 108.6)
- moved R12 50.4 mm to (105.2, 126.6), turned to 180 degrees
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Connections:
- net /current_sensor2/VIN+ renamed /24_IN_PMM
- net /current_sensor3/VIN- renamed /24V_OUT
- C5 pad 1: /current_sensor2/3V3 -> 3.3V
- C5 pad 2: /current_sensor2/GND -> A_GND
- C6 pad 1: /current_sensor3/3V3 -> 3.3V
- C6 pad 2: /current_sensor3/GND -> A_GND
- Cin1 pad 1: 24V -> /24V_IN
- Cinx1 pad 1: 24V -> /24V_IN
- Q1 pad 1: /LMG5200/high_side_FET -> /24V_IN
- R1 pad 1: /cap_volt -> Net-(D2-A)
- R1 pad 2: /LMG5200/cap_volt_pico_adc -> /Pico/LED0
- R10 pad 1: /current_sensor3/3V3 -> 3.3V
- R10 pad 2: /current_sensor3/SCL -> /I2C_current_SCL
- R11 pad 1: /current_sensor3/3V3 -> 3.3V
- R11 pad 2: /current_sensor3/SDA -> /I2C_current_SDA
- R12 pad 1: /current_sensor3/3V3 -> 3.3V
- R15 pad 1: /LMG5200/cap_volt_pico_adc -> Net-(D1-A)
- R15 pad 2: P_GND -> /Pico/LED1
- R5 pad 2: /current_sensor2/VIN- -> /24V_IN
- R6 pad 1: /current_sensor2/3V3 -> 3.3V
- R6 pad 2: /current_sensor2/SCL -> /I2C_current_SCL
- R7 pad 1: /current_sensor2/3V3 -> 3.3V
- R7 pad 2: /current_sensor2/SDA -> /I2C_current_SDA
- R8 pad 1: /current_sensor2/3V3 -> 3.3V
- R9 pad 1: /current_sensor3/VIN+ -> /24V_IN
- U1 pad 3: 24V -> /24V_IN
- U1 pad 5: 24V -> /24V_IN
- U3 pad 1: /current_sensor2/GND -> A_GND
- U3 pad 3: /current_sensor2/SDA -> /I2C_current_SDA
- U3 pad 4: /current_sensor2/SCL -> /I2C_current_SCL
- U3 pad 5: /current_sensor2/3V3 -> 3.3V
- U3 pad 6: /current_sensor2/GND -> A_GND
- U3 pad 7: /current_sensor2/VIN- -> /24V_IN
- U4 pad 2: /current_sensor3/GND -> A_GND
- U4 pad 3: /current_sensor3/SDA -> /I2C_current_SDA
- U4 pad 4: /current_sensor3/SCL -> /I2C_current_SCL
- U4 pad 5: /current_sensor3/3V3 -> 3.3V
- U4 pad 6: /current_sensor3/GND -> A_GND
- U4 pad 8: /current_sensor3/VIN+ -> /24V_IN
- U5 pad 31: /Pico/ADC_0 -> unconnected-(U5-GP26-Pad31)
- U5 pad 32: /Pico/ADC_1 -> unconnected-(U5-GP27-Pad32)
- U5 pad 34: /Pico/ADC_2 -> unconnected-(U5-GP28-Pad34)
Routing:
- net 24V: track 4.29 -> 0.00 mm
- net /24V_IN: track 0.00 -> 4.29 mm
- net (no net): vias 0 -> 20
