File: Design Files/Controller Board V1/current_sensor1.kicad_sch (KiCad schematic)
At the start: 5 parts, among them U2 INA219BIDR

Commit message: general layout revised
goodnight
Parts:
- R2: footprint Resistor_SMD:R_0805_2012Metric -> Resistor_SMD:R_2512_6332Metric
Changed lines of the file:
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@@
 			)
 		)
-		(property "Footprint" "Resistor_SMD:R_0805_2012Metric"
+		(property "Footprint" "Resistor_SMD:R_2512_6332Metric"
 			(at 139.7 80.518 90)
 			(effects

Commit message: Minor Changes
Connections:
- net 3V3: no longer C4.1, U2.5 (VS)
- new net 5V: C4.1, U2.5 (VS)
Changed lines of the file:
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@@
 		(shape input)
 		(at 120.65 110.49 270)
+		(fields_autoplaced yes)
 		(effects
 			(font
@@
 		(shape input)
 		(at 134.62 71.12 90)
+		(fields_autoplaced yes)
 		(effects
 			(font
@@
 		(shape input)
 		(at 158.75 74.93 90)
+		(fields_autoplaced yes)
 		(effects
 			(font
@@
 		(shape output)
 		(at 176.53 90.17 0)
+		(fields_autoplaced yes)
 		(effects
 			(font
@@
 		)
 	)
-	(hierarchical_label "3V3"
+	(hierarchical_label "5V"
 		(shape input)
 		(at 120.65 85.09 90)
+		(fields_autoplaced yes)
 		(effects
 			(font
@@
 		(shape input)
 		(at 158.75 110.49 270)
+		(fields_autoplaced yes)
 		(effects
 			(font
@@
 		(shape input)
 		(at 144.78 71.12 90)
+		(fields_autoplaced yes)
 		(effects
 			(font
@@
 		(shape output)
 		(at 176.53 95.25 0)
+		(fields_autoplaced yes)
 		(effects
 			(font

Commit message: OOps, pushing late
Connections:
- net 3V3 is gone; now on net 5V: R3.1, R4.1
Changed lines of the file:
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@@
-		)
-	)
-	(hierarchical_label "3V3"
-		(shape input)
-		(at 158.75 74.93 90)
-		(fields_autoplaced yes)
-		(effects
-			(font
-				(size 1.27 1.27)
-			)
-			(justify left)
 		)
 	)
@@
 		)
 	)
+	(hierarchical_label "5V"
+		(shape input)
+		(at 158.75 74.93 90)
+		(fields_autoplaced yes)
+		(effects
+			(font
+				(size 1.27 1.27)
+			)
+			(justify left)
+		)
+	)
