File: Design Files/Controller Board V1/current_sensor2.kicad_sch (KiCad schematic)
At the start: 6 parts, among them U3 INA219BIDR

Commit message: general layout revised
goodnight
Parts:
- R5: footprint Resistor_SMD:R_0805_2012Metric -> Resistor_SMD:R_2512_6332Metric
Changed lines of the file:
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@@
 			)
 		)
-		(property "Footprint" "Resistor_SMD:R_0805_2012Metric"
+		(property "Footprint" "Resistor_SMD:R_2512_6332Metric"
 			(at 135.89 94.488 90)
 			(effects

Commit message: Minor Changes
Connections:
- net 3V3: no longer C5.1, U3.5 (VS)
- new net 5V: C5.1, U3.5 (VS)
Changed lines of the file:
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@@
 		(shape input)
 		(at 116.84 124.46 270)
+		(fields_autoplaced yes)
 		(effects
 			(font
@@
 		(shape input)
 		(at 154.94 88.9 90)
+		(fields_autoplaced yes)
 		(effects
 			(font
@@
 		)
 	)
-	(hierarchical_label "3V3"
+	(hierarchical_label "5V"
 		(shape input)
 		(at 116.84 99.06 90)
+		(fields_autoplaced yes)
 		(effects
 			(font
@@
 		(shape output)
 		(at 172.72 104.14 0)
+		(fields_autoplaced yes)
 		(effects
 			(font
@@
 		(shape output)
 		(at 172.72 109.22 0)
+		(fields_autoplaced yes)
 		(effects
 			(font
@@
 		(shape input)
 		(at 140.97 85.09 90)
+		(fields_autoplaced yes)
 		(effects
 			(font
@@
 		(shape input)
 		(at 154.94 124.46 270)
+		(fields_autoplaced yes)
 		(effects
 			(font
@@
 		(shape input)
 		(at 130.81 85.09 90)
+		(fields_autoplaced yes)
 		(effects
 			(font

Commit message: OOps, pushing late
Connections:
- net 3V3 is gone; now on net 5V: R6.1, R7.1, R8.1
Changed lines of the file:
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@@
-		)
-	)
-	(hierarchical_label "3V3"
-		(shape input)
-		(at 154.94 88.9 90)
-		(fields_autoplaced yes)
-		(effects
-			(font
-				(size 1.27 1.27)
-			)
-			(justify left)
 		)
 	)
@@
 		)
 	)
+	(hierarchical_label "5V"
+		(shape input)
+		(at 154.94 88.9 90)
+		(fields_autoplaced yes)
+		(effects
+			(font
+				(size 1.27 1.27)
+			)
+			(justify left)
+		)
+	)
