File: Design Files/Controller Board V1/current_sensor3.kicad_sch (KiCad schematic)
At the start: 6 parts, among them U4 INA219BIDR

Commit message: general layout revised
goodnight
Parts:
- R9: footprint Resistor_SMD:R_0805_2012Metric -> Resistor_SMD:R_2512_6332Metric
Changed lines of the file:
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@@
 			)
 		)
-		(property "Footprint" "Resistor_SMD:R_0805_2012Metric"
+		(property "Footprint" "Resistor_SMD:R_2512_6332Metric"
 			(at 139.7 84.328 90)
 			(effects

Commit message: Minor Changes
Connections:
- net 3V3: no longer C6.1, U4.5 (VS)
- new net 5V: C6.1, U4.5 (VS)
Changed lines of the file:
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@@
 		)
 	)
-	(hierarchical_label "3V3"
+	(hierarchical_label "5V"
 		(shape input)
 		(at 120.65 88.9 90)
+		(fields_autoplaced yes)
 		(effects
 			(font
@@
 		(shape output)
 		(at 176.53 99.06 0)
+		(fields_autoplaced yes)
 		(effects
 			(font
@@
 		(shape input)
 		(at 158.75 114.3 270)
+		(fields_autoplaced yes)
 		(effects
 			(font
@@
 		(shape input)
 		(at 158.75 78.74 90)
+		(fields_autoplaced yes)
 		(effects
 			(font
@@
 		(shape input)
 		(at 134.62 74.93 90)
+		(fields_autoplaced yes)
 		(effects
 			(font
@@
 		(shape input)
 		(at 120.65 114.3 270)
+		(fields_autoplaced yes)
 		(effects
 			(font
@@
 		(shape output)
 		(at 176.53 93.98 0)
+		(fields_autoplaced yes)
 		(effects
 			(font
@@
 		(shape input)
 		(at 144.78 74.93 90)
+		(fields_autoplaced yes)
 		(effects
 			(font

Commit message: OOps, pushing late
Parts:
- C6: footprint Capacitor_SMD:C_0603_1608Metric -> PGA460TW:C_0603_1608Metric
- R10, R11, R12: footprint Resistor_SMD:R_0603_1608Metric -> PGA460TW:R_0603_1608Metric
Connections:
- net 3V3 is gone; now on net 5V: R10.1, R11.1, R12.1
Changed lines of the file:
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@@
-		)
-	)
-	(hierarchical_label "3V3"
-		(shape input)
-		(at 158.75 78.74 90)
-		(fields_autoplaced yes)
-		(effects
-			(font
-				(size 1.27 1.27)
-			)
-			(justify left)
 		)
 	)
@@
 			)
 			(justify right)
+		)
+	)
+	(hierarchical_label "5V"
+		(shape input)
+		(at 158.75 78.74 90)
+		(fields_autoplaced yes)
+		(effects
+			(font
+				(size 1.27 1.27)
+			)
+			(justify left)
 		)
 	)
@@
 			)
 		)
-		(property "Footprint" "Resistor_SMD:R_0603_1608Metric"
+		(property "Footprint" "PGA460TW:R_0603_1608Metric"
 			(at 169.672 88.9 90)
 			(effects
@@
 			)
 		)
-		(property "Footprint" "Resistor_SMD:R_0603_1608Metric"
+		(property "Footprint" "PGA460TW:R_0603_1608Metric"
 			(at 163.322 88.9 90)
 			(effects
@@
 			)
 		)
-		(property "Footprint" "Capacitor_SMD:C_0603_1608Metric"
+		(property "Footprint" "PGA460TW:C_0603_1608Metric"
 			(at 121.6152 105.41 0)
 			(effects
@@
 			)
 		)
-		(property "Footprint" "Resistor_SMD:R_0603_1608Metric"
+		(property "Footprint" "PGA460TW:R_0603_1608Metric"
 			(at 156.972 88.9 90)
 			(effects
