File: Design Files/Controller Board V1/LMG5200.kicad_sch (KiCad schematic)
At the start: 8 parts, among them Q1 LMG5200

Commit message: Ready For Design Review
Connections:
- net D_GND: no longer C2.2
- net P_GND: now also C2.2
Changed lines of the file:
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@@
 			)
 		)
-		(property "Value" "D_GND"
+		(property "Value" "P_GND"
 			(at 108.204 83.82 0)
 			(effects

Commit message: Last second changes
Connections:
- net GND is gone; now on net P_GND: C12.1
Changed lines of the file:
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@@
 		(shape input)
 		(at 158.75 97.79 0)
-		(fields_autoplaced yes)
 		(effects
 			(font
@@
 		(shape input)
 		(at 120.65 80.01 90)
-		(fields_autoplaced yes)
 		(effects
 			(font
@@
 		(shape input)
 		(at 110.49 100.33 180)
-		(fields_autoplaced yes)
 		(effects
 			(font
@@
 		(shape input)
 		(at 88.9 97.79 180)
-		(fields_autoplaced yes)
 		(effects
 			(font
@@
 		(shape input)
 		(at 125.73 85.09 90)
-		(fields_autoplaced yes)
 		(effects
 			(font
@@
 			)
 		)
-		(property "Value" "GND"
+		(property "Value" "P_GND"
 			(at 144.272 85.09 0)
 			(effects

Commit message: changes
Connections:
- net high_side_FET: now also C12.2
Changed lines of the file:
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@@
 	(wire
 		(pts
-			(xy 125.73 86.36) (xy 132.08 86.36)
+			(xy 127 86.36) (xy 132.08 86.36)
+		)
+		(stroke
+			(width 0)
+			(type default)
+		)
+	)
+	(wire
+		(pts
+			(xy 125.73 85.09) (xy 127 85.09)
 		)
 		(stroke
@@
 		)
 		(stroke
+			(width 0)
+			(type default)
+		)
+	)
+	(wire
+		(pts
+			(xy 127 85.09) (xy 127 86.36)
+		)
+		(stroke
